File: HB-LC-DimPWM-PCB.kicad_pcb (KiCad board)
At the start: 2 copper layers, 168.2 x 57 mm, 233 parts, among them J1 SWD, J3 Conn_01x04_Male, Q1 S9013, Q10 BSS84, Q11 2N7002, Q12 BSS84, Q13 2N7002, Q14 VS5810AS, Q15 VS5810AS, Q16 VS5810AS, Q2 BSS84, Q3 2N7002, Q4 VS5810AS, Q5 S9013, Q6 S9013, Q7 S9013, Q8 BSS84, Q9 2N7002, U1 STM32F103C8Tx, U2 AMS1117-3.3, U3 HomeMatic-sensor, Y1 8MHz

Commit message: Finish layout of first four dimmer channels
Parts:
- removed the C13 at (148.5, 66.2)
- removed the C13 at (148.5, 93.8)
- removed the C13 at (196.7, 114.5)
- removed the C14 at (148.5, 73.0)
- removed the C14 at (148.5, 100.6)
- removed the C14 at (196.7, 107.7)
- removed the C15 at (148.5, 79.8)
- removed the C15 at (148.5, 107.4)
- removed the C15 at (196.7, 100.9)
- removed the C16 at (148.6, 86.7)
- removed the C16 at (148.6, 114.2)
- removed the C16 at (196.7, 94.0)
- removed the C17 at (136.2, 64.2)
- removed the C17 at (136.2, 91.8)
- removed the C17 at (209.0, 116.5)
- removed the C18 at (123.8, 76.4)
- removed the C18 at (123.8, 104.0)
- removed the C18 at (221.4, 104.3)
- removed the C19 at (129.2, 76.4)
- removed the C19 at (129.2, 104.0)
- removed the C19 at (216.0, 104.3)
- removed the C20 at (136.3, 89.0)
- removed the C20 at (136.3, 116.6)
- removed the C20 at (208.9, 91.7)
- removed the C21 at (93.3, 64.3)
- removed the C21 at (93.3, 91.9)
- removed the C21 at (251.9, 116.4)
- removed the C22 at (116.2, 76.4)
- removed the C22 at (116.2, 104.0)
- removed the C22 at (229.0, 104.3)
- removed the C23 at (109.1, 76.4)
- removed the C23 at (109.1, 104.0)
- removed the C23 at (236.1, 104.3)
- removed the C24 at (93.3, 88.4)
- removed the C24 at (93.3, 116.0)
- removed the C24 at (251.9, 92.3)
- removed the F2 at (101.0, 67.2)
- removed the F2 at (101.0, 94.8)
- removed the F2 at (244.2, 113.5)
- removed the F3 at (101.0, 73.3)
- removed the F3 at (101.0, 100.9)
- removed the F3 at (244.2, 107.4)
- removed the F4 at (101.0, 79.4)
- removed the F4 at (101.0, 107.0)
- removed the F4 at (244.2, 101.3)
- removed the F5 at (101.0, 85.5)
- removed the F5 at (101.0, 113.1)
- removed the F5 at (244.2, 95.2)
- removed the J3 at (93.3, 68.8)
- removed the J3 at (93.3, 96.4)
- removed the J3 at (251.9, 111.9)
- removed the L1 at (112.7, 68.7)
- removed the L1 at (112.7, 96.3)
- removed the L1 at (232.5, 112.0)
- removed the L2 at (126.4, 68.7)
- removed the L2 at (126.4, 96.3)
- removed the L2 at (218.8, 112.0)
- removed the L3 at (126.3, 84.1)
- removed the L3 at (126.3, 111.7)
- removed the L3 at (218.9, 96.6)
- removed the L4 at (112.6, 84.1)
- removed the L4 at (112.6, 111.7)
- removed the L4 at (232.6, 96.6)
- removed the Q1 at (146.2, 68.0)
- removed the Q1 at (146.2, 95.6)
- removed the Q1 at (199.0, 112.7)
- removed the Q10 at (146.2, 78.2)
- removed the Q10 at (146.2, 105.8)
- removed the Q10 at (199.0, 102.5)
- removed the Q11 at (142.7, 81.6)
- removed the Q11 at (142.7, 109.2)
- removed the Q11 at (202.5, 99.1)
- removed the Q12 at (146.2, 85.0)
- removed the Q12 at (146.2, 112.6)
- removed the Q12 at (199.0, 95.7)
- removed the Q13 at (142.7, 88.4)
- removed the Q13 at (142.7, 116.0)
- removed the Q13 at (202.5, 92.3)
- removed the Q14 at (137.1, 73.8)
- removed the Q14 at (137.1, 101.4)
- removed the Q14 at (208.1, 106.9)
- removed the Q15 at (137.1, 79.3)
- removed the Q15 at (137.1, 106.9)
- removed the Q15 at (208.1, 101.4)
- removed the Q16 at (137.1, 84.8)
- removed the Q16 at (137.1, 112.4)
- removed the Q16 at (208.1, 95.9)
- removed the Q2 at (146.2, 64.6)
- removed the Q2 at (146.2, 92.2)
- removed the Q2 at (199.0, 116.1)
- removed the Q3 at (142.7, 68.0)
- removed the Q3 at (142.7, 95.6)
- removed the Q3 at (202.5, 112.7)
- removed the Q4 at (137.1, 68.3)
- removed the Q4 at (137.1, 95.9)
- removed the Q4 at (208.1, 112.4)
- removed the Q5 at (146.2, 74.8)
- removed the Q5 at (146.2, 102.4)
- removed the Q5 at (199.0, 105.9)
- removed the Q6 at (146.2, 81.6)
- removed the Q6 at (146.2, 109.2)
- removed the Q6 at (199.0, 99.1)
- removed the Q7 at (146.2, 88.4)
- removed the Q7 at (146.2, 116.0)
- removed the Q7 at (199.0, 92.3)
- removed the Q8 at (146.2, 71.4)
- removed the Q8 at (146.2, 99.0)
- removed the Q8 at (199.0, 109.3)
- removed the Q9 at (142.7, 74.8)
- removed the Q9 at (142.7, 102.4)
- removed the Q9 at (202.5, 105.9)
- removed the R10 at (148.6, 88.7)
- removed the R10 at (148.6, 116.2)
- removed the R10 at (196.7, 92.0)
- removed the R11 at (148.5, 71.0)
- removed the R11 at (148.5, 98.6)
- removed the R11 at (196.7, 109.7)
- removed the R12 at (148.5, 77.8)
- removed the R12 at (148.5, 105.4)
- removed the R12 at (196.7, 102.9)
- removed the R13 at (148.6, 84.7)
- removed the R13 at (148.6, 112.2)
- removed the R13 at (196.7, 96.0)
- removed the R14 at (142.6, 70.6)
- removed the R14 at (142.6, 98.2)
- removed the R14 at (202.6, 110.1)
- removed the R15 at (142.6, 72.2)
- removed the R15 at (142.6, 99.8)
- removed the R15 at (202.6, 108.5)
- removed the R16 at (142.7, 77.4)
- removed the R16 at (142.7, 105.0)
- removed the R16 at (202.5, 103.3)
- removed the R17 at (142.7, 79.0)
- removed the R17 at (142.7, 106.6)
- removed the R17 at (202.5, 101.7)
- removed the R18 at (142.6, 84.2)
- removed the R18 at (142.6, 111.8)
- removed the R18 at (202.6, 96.5)
- removed the R19 at (142.6, 85.8)
- removed the R19 at (142.6, 113.4)
- removed the R19 at (202.6, 94.9)
- removed the R4 at (148.5, 68.2)
- removed the R4 at (148.5, 95.8)
- removed the R4 at (196.7, 112.5)
- removed the R5 at (148.5, 64.2)
- removed the R5 at (148.5, 91.8)
- removed the R5 at (196.7, 116.5)
- removed the R6 at (142.6, 63.8)
- removed the R6 at (142.6, 91.4)
- removed the R6 at (202.6, 116.9)
- removed the R7 at (142.6, 65.3)
- removed the R7 at (142.6, 92.9)
- removed the R7 at (202.6, 115.4)
- removed the R8 at (148.5, 75.0)
- removed the R8 at (148.5, 102.6)
- removed the R8 at (196.7, 105.7)
- removed the R9 at (148.5, 81.8)
- removed the R9 at (148.5, 109.4)
- removed the R9 at (196.7, 98.9)
- added C25: 1uF, Capacitor_SMD:C_0402_1005Metric, F.Cu at (440.3, 29.7)
- added C26: 1uF, Capacitor_SMD:C_0402_1005Metric, F.Cu at (447.8, 25.1)
- added C27: 1uF, Capacitor_SMD:C_0402_1005Metric, F.Cu at (448.3, 22.1)
- added C28: 1uF, Capacitor_SMD:C_0402_1005Metric, F.Cu at (443.8, 27.7)
- added C29: 100p, Capacitor_SMD:C_0805_2012Metric, F.Cu at (449.9, 14.6)
- added C30: 100p, Capacitor_SMD:C_0805_2012Metric, F.Cu at (462.6, 2.86)
- added C31: 100p, Capacitor_SMD:C_0805_2012Metric, F.Cu at (459.9, -0.09)
- added C32: 100p, Capacitor_SMD:C_0805_2012Metric, F.Cu at (432.6, 29.4)
- added C33: 1uF, Capacitor_SMD:C_1206_3216Metric, F.Cu at (460.5, -3.21)
- added C34: 1uF, Capacitor_SMD:C_1206_3216Metric, F.Cu at (423.2, 28.1)
- added C35: 1uF, Capacitor_SMD:C_1206_3216Metric, F.Cu at (431.6, 15.9)
- added C36: 1uF, Capacitor_SMD:C_1206_3216Metric, F.Cu at (417.6, 28.1)
- added C37: 1uF, Capacitor_SMD:C_0402_1005Metric, F.Cu at (356.4, 129.0)
- added C38: 1uF, Capacitor_SMD:C_0402_1005Metric, F.Cu at (352.4, 134.0)
- added C39: 1uF, Capacitor_SMD:C_0402_1005Metric, F.Cu at (338.4, 148.8)
- added C40: 1uF, Capacitor_SMD:C_0402_1005Metric, F.Cu at (342.9, 143.2)
- added C41: 100p, Capacitor_SMD:C_0805_2012Metric, F.Cu at (354.5, 121.0)
- added C42: 100p, Capacitor_SMD:C_0805_2012Metric, F.Cu at (327.2, 150.5)
- added C43: 100p, Capacitor_SMD:C_0805_2012Metric, F.Cu at (357.1, 124.0)
- added C44: 100p, Capacitor_SMD:C_0805_2012Metric, F.Cu at (344.5, 135.8)
- added C45: 1uF, Capacitor_SMD:C_1206_3216Metric, F.Cu at (317.8, 149.2)
- added C46: 1uF, Capacitor_SMD:C_1206_3216Metric, F.Cu at (355.1, 117.9)
- added C47: 1uF, Capacitor_SMD:C_1206_3216Metric, F.Cu at (326.1, 137.0)
- added C48: 1uF, Capacitor_SMD:C_1206_3216Metric, F.Cu at (312.1, 149.2)
- added C49: 1uF, Capacitor_SMD:C_0402_1005Metric, F.Cu at (381.9, 112.2)
- added C50: 1uF, Capacitor_SMD:C_0402_1005Metric, F.Cu at (384.8, 112.2)
- added C51: 1uF, Capacitor_SMD:C_0402_1005Metric, F.Cu at (394.7, 108.3)
- added C52: 1uF, Capacitor_SMD:C_0402_1005Metric, F.Cu at (379.0, 112.2)
- added C53: 100p, Capacitor_SMD:C_0805_2012Metric, F.Cu at (412.7, 96.1)
- added C54: 100p, Capacitor_SMD:C_0805_2012Metric, F.Cu at (425.4, 84.3)
- added C55: 100p, Capacitor_SMD:C_0805_2012Metric, F.Cu at (422.7, 81.3)
- added C56: 100p, Capacitor_SMD:C_0805_2012Metric, F.Cu at (395.4, 110.8)
- added C57: 1uF, Capacitor_SMD:C_1206_3216Metric, F.Cu at (394.4, 97.4)
- added C58: 1uF, Capacitor_SMD:C_1206_3216Metric, F.Cu at (386.0, 109.5)
- added C59: 1uF, Capacitor_SMD:C_1206_3216Metric, F.Cu at (423.3, 78.2)
- added C60: 1uF, Capacitor_SMD:C_1206_3216Metric, F.Cu at (380.4, 109.5)
- added F10: 15V 5A, Fuse:Fuse_2920_7451Metric, F.Cu at (336.9, 119.8)
- added F11: 15V 5A, Fuse:Fuse_2920_7451Metric, F.Cu at (314.5, 144.1)
- added F12: 15V 5A, Fuse:Fuse_2920_7451Metric, F.Cu at (328.5, 131.9)
- added F13: 15V 5A, Fuse:Fuse_2920_7451Metric, F.Cu at (347.2, 119.8)
- added F14: 15V 5A, Fuse:Fuse_2920_7451Metric, F.Cu at (405.2, 80.1)
- added F15: 15V 5A, Fuse:Fuse_2920_7451Metric, F.Cu at (382.7, 104.4)
- added F16: 15V 5A, Fuse:Fuse_2920_7451Metric, F.Cu at (396.7, 92.2)
- added F17: 15V 5A, Fuse:Fuse_2920_7451Metric, F.Cu at (415.4, 80.1)
- added F6: 15V 5A, Fuse:Fuse_2920_7451Metric, F.Cu at (419.9, 22.9)
- added F7: 15V 5A, Fuse:Fuse_2920_7451Metric, F.Cu at (442.4, -1.35)
- added F8: 15V 5A, Fuse:Fuse_2920_7451Metric, F.Cu at (433.9, 10.8)
- added F9: 15V 5A, Fuse:Fuse_2920_7451Metric, F.Cu at (452.6, -1.35)
- added J4: Conn_01x04_Male, Connector_Phoenix_MC_HighVoltage:PhoenixContact_MC_1,5_4-G-5.08_1x04_P5.08mm_Horizontal, F.Cu at (404.4, -1.70)
- added J5: Conn_01x04_Male, Connector_Phoenix_MC_HighVoltage:PhoenixContact_MC_1,5_4-G-5.08_1x04_P5.08mm_Horizontal, F.Cu at (299.0, 119.4)
- added J6: Conn_01x04_Male, Connector_Phoenix_MC_HighVoltage:PhoenixContact_MC_1,5_4-G-5.08_1x04_P5.08mm_Horizontal, F.Cu at (367.2, 79.7)
- added L10: 3.3uH, Inductor_Sunlord:SMD-PIND-10.5x11.5x4_2.5x3.0, F.Cu at (302.3, 146.6)
- added L11: 3.3uH, Inductor_Sunlord:SMD-PIND-10.5x11.5x4_2.5x3.0, F.Cu at (324.8, 122.3)
- added L12: 3.3uH, Inductor_Sunlord:SMD-PIND-10.5x11.5x4_2.5x3.0, F.Cu at (302.3, 134.5)
- added L13: 3.3uH, Inductor_Sunlord:SMD-PIND-10.5x11.5x4_2.5x3.0, F.Cu at (393.0, 82.6)
- added L14: 3.3uH, Inductor_Sunlord:SMD-PIND-10.5x11.5x4_2.5x3.0, F.Cu at (370.6, 106.9)
- added L15: 3.3uH, Inductor_Sunlord:SMD-PIND-10.5x11.5x4_2.5x3.0, F.Cu at (384.6, 94.8)
- added L16: 3.3uH, Inductor_Sunlord:SMD-PIND-10.5x11.5x4_2.5x3.0, F.Cu at (370.6, 94.8)
- added L5: 3.3uH, Inductor_Sunlord:SMD-PIND-10.5x11.5x4_2.5x3.0, F.Cu at (407.8, 13.4)
- added L6: 3.3uH, Inductor_Sunlord:SMD-PIND-10.5x11.5x4_2.5x3.0, F.Cu at (407.8, 25.5)
- added L7: 3.3uH, Inductor_Sunlord:SMD-PIND-10.5x11.5x4_2.5x3.0, F.Cu at (421.8, 13.4)
- added L8: 3.3uH, Inductor_Sunlord:SMD-PIND-10.5x11.5x4_2.5x3.0, F.Cu at (430.2, 1.21)
- added L9: 3.3uH, Inductor_Sunlord:SMD-PIND-10.5x11.5x4_2.5x3.0, F.Cu at (316.3, 134.5)
- added Q17: S9013, Package_TO_SOT_SMD:SOT-23, F.Cu at (436.6, 16.6)
- added Q18: S9013, Package_TO_SOT_SMD:SOT-23, F.Cu at (428.2, 28.2)
- added Q19: S9013, Package_TO_SOT_SMD:SOT-23, F.Cu at (435.7, 21.1)
- added Q20: S9013, Package_TO_SOT_SMD:SOT-23, F.Cu at (449.7, 10.9)
- added Q21: BSS84, Package_TO_SOT_SMD:SOT-23, F.Cu at (441.0, 17.3)
- added Q22: 2N7002, Package_TO_SOT_SMD:SOT-23, F.Cu at (435.7, 25.6)
- added Q23: BSS84, Package_TO_SOT_SMD:SOT-23, F.Cu at (458.1, 4.43)
- added Q24: 2N7002, Package_TO_SOT_SMD:SOT-23, F.Cu at (444.6, 21.9)
- added Q25: BSS84, Package_TO_SOT_SMD:SOT-23, F.Cu at (440.1, 26.4)
- added Q26: 2N7002, Package_TO_SOT_SMD:SOT-23, F.Cu at (454.1, 10.9)
- added Q27: BSS84, Package_TO_SOT_SMD:SOT-23, F.Cu at (440.1, 21.9)
- added Q28: 2N7002, Package_TO_SOT_SMD:SOT-23, F.Cu at (445.5, 17.3)
- added Q29: VS5810AS, Package_SO:SOIC-8_3.9x4.9mm_P1.27mm, F.Cu at (443.2, 11.8)
- added Q30: VS5810AS, Package_SO:SOIC-8_3.9x4.9mm_P1.27mm, F.Cu at (451.7, 5.38)
- added Q31: VS5810AS, Package_SO:SOIC-8_3.9x4.9mm_P1.27mm, F.Cu at (429.2, 22.7)
- added Q32: VS5810AS, Package_SO:SOIC-8_3.9x4.9mm_P1.27mm, F.Cu at (443.2, 5.38)
- added Q33: S9013, Package_TO_SOT_SMD:SOT-23, F.Cu at (331.2, 137.7)
- added Q34: S9013, Package_TO_SOT_SMD:SOT-23, F.Cu at (330.3, 146.8)
- added Q35: S9013, Package_TO_SOT_SMD:SOT-23, F.Cu at (340.1, 138.4)
- added Q36: S9013, Package_TO_SOT_SMD:SOT-23, F.Cu at (352.7, 125.5)
- added Q37: BSS84, Package_TO_SOT_SMD:SOT-23, F.Cu at (334.7, 147.6)
- added Q38: 2N7002, Package_TO_SOT_SMD:SOT-23, F.Cu at (348.7, 132.0)
- added Q39: BSS84, Package_TO_SOT_SMD:SOT-23, F.Cu at (339.2, 143.0)
- added Q40: 2N7002, Package_TO_SOT_SMD:SOT-23, F.Cu at (335.6, 138.4)
- added Q41: BSS84, Package_TO_SOT_SMD:SOT-23, F.Cu at (344.3, 132.0)
- added Q42: 2N7002, Package_TO_SOT_SMD:SOT-23, F.Cu at (330.3, 142.2)
- added Q43: BSS84, Package_TO_SOT_SMD:SOT-23, F.Cu at (322.8, 149.3)
- added Q44: 2N7002, Package_TO_SOT_SMD:SOT-23, F.Cu at (334.7, 143.0)
- added Q45: VS5810AS, Package_SO:SOIC-8_3.9x4.9mm_P1.27mm, F.Cu at (323.8, 143.8)
- added Q46: VS5810AS, Package_SO:SOIC-8_3.9x4.9mm_P1.27mm, F.Cu at (337.8, 126.5)
- added Q47: VS5810AS, Package_SO:SOIC-8_3.9x4.9mm_P1.27mm, F.Cu at (346.3, 126.5)
- added Q48: VS5810AS, Package_SO:SOIC-8_3.9x4.9mm_P1.27mm, F.Cu at (337.8, 132.9)
- added Q49: S9013, Package_TO_SOT_SMD:SOT-23, F.Cu at (399.4, 98.0)
- added Q50: S9013, Package_TO_SOT_SMD:SOT-23, F.Cu at (391.0, 109.6)
- added Q51: S9013, Package_TO_SOT_SMD:SOT-23, F.Cu at (398.5, 102.5)
- added Q52: S9013, Package_TO_SOT_SMD:SOT-23, F.Cu at (407.4, 103.3)
- added Q53: BSS84, Package_TO_SOT_SMD:SOT-23, F.Cu at (416.9, 92.3)
- added Q54: 2N7002, Package_TO_SOT_SMD:SOT-23, F.Cu at (402.9, 103.3)
- added Q55: BSS84, Package_TO_SOT_SMD:SOT-23, F.Cu at (408.3, 98.8)
- added Q56: 2N7002, Package_TO_SOT_SMD:SOT-23, F.Cu at (398.5, 107.1)
- added Q57: BSS84, Package_TO_SOT_SMD:SOT-23, F.Cu at (420.9, 85.9)
- added Q58: 2N7002, Package_TO_SOT_SMD:SOT-23, F.Cu at (403.8, 98.8)
- added Q59: BSS84, Package_TO_SOT_SMD:SOT-23, F.Cu at (412.5, 92.3)
- added Q60: 2N7002, Package_TO_SOT_SMD:SOT-23, F.Cu at (402.9, 107.9)
- added Q61: VS5810AS, Package_SO:SOIC-8_3.9x4.9mm_P1.27mm, F.Cu at (406.0, 93.3)
- added Q62: VS5810AS, Package_SO:SOIC-8_3.9x4.9mm_P1.27mm, F.Cu at (414.5, 86.8)
- added Q63: VS5810AS, Package_SO:SOIC-8_3.9x4.9mm_P1.27mm, F.Cu at (406.0, 86.8)
- added Q64: VS5810AS, Package_SO:SOIC-8_3.9x4.9mm_P1.27mm, F.Cu at (392.0, 104.1)
- added R20: 10k, Resistor_SMD:R_0402_1005Metric, F.Cu at (419.1, 30.7)
- added R21: 10k, Resistor_SMD:R_0402_1005Metric, F.Cu at (422.0, 30.7)
- added R22: 10k, Resistor_SMD:R_0402_1005Metric, F.Cu at (431.9, 26.9)
- added R23: 10k, Resistor_SMD:R_0402_1005Metric, F.Cu at (416.2, 30.7)
- added R24: 1k, Resistor_SMD:R_0402_1005Metric, F.Cu at (463.6, -0.57)
- added R25: 1k, Resistor_SMD:R_0402_1005Metric, F.Cu at (453.2, 17.1)
- added R26: 1k, Resistor_SMD:R_0402_1005Metric, F.Cu at (461.8, 7.84)
- added R27: 1k, Resistor_SMD:R_0402_1005Metric, F.Cu at (457.8, 12.9)
- added R28: 22R, Resistor_SMD:R_0603_1608Metric, F.Cu at (444.4, 25.4)
- added R29: 22R, Resistor_SMD:R_0603_1608Metric, F.Cu at (458.4, 8.10)
- added R30: 22R, Resistor_SMD:R_0603_1608Metric, F.Cu at (462.4, 5.59)
- added R31: 22R, Resistor_SMD:R_0603_1608Metric, F.Cu at (458.4, 10.6)
- added R32: 22R, Resistor_SMD:R_0603_1608Metric, F.Cu at (449.7, 17.4)
- added R33: 22R, Resistor_SMD:R_0603_1608Metric, F.Cu at (436.8, 30.0)
- added R34: 22R, Resistor_SMD:R_0603_1608Metric, F.Cu at (454.1, 14.4)
- added R35: 22R, Resistor_SMD:R_0603_1608Metric, F.Cu at (449.7, 19.9)
- added R36: 10k, Resistor_SMD:R_0402_1005Metric, F.Cu at (326.5, 148.0)
- added R37: 10k, Resistor_SMD:R_0402_1005Metric, F.Cu at (316.6, 151.9)
- added R38: 10k, Resistor_SMD:R_0402_1005Metric, F.Cu at (313.7, 151.9)
- added R39: 10k, Resistor_SMD:R_0402_1005Metric, F.Cu at (310.8, 151.9)
- added R40: 1k, Resistor_SMD:R_0402_1005Metric, F.Cu at (347.8, 138.2)
- added R41: 1k, Resistor_SMD:R_0402_1005Metric, F.Cu at (334.9, 150.8)
- added R42: 1k, Resistor_SMD:R_0402_1005Metric, F.Cu at (342.4, 146.3)
- added R43: 1k, Resistor_SMD:R_0402_1005Metric, F.Cu at (358.2, 120.5)
- added R44: 22R, Resistor_SMD:R_0603_1608Metric, F.Cu at (331.4, 151.1)
- added R45: 22R, Resistor_SMD:R_0603_1608Metric, F.Cu at (344.3, 138.5)
- added R46: 22R, Resistor_SMD:R_0603_1608Metric, F.Cu at (348.7, 135.5)
- added R47: 22R, Resistor_SMD:R_0603_1608Metric, F.Cu at (344.3, 141.0)
- added R48: 22R, Resistor_SMD:R_0603_1608Metric, F.Cu at (352.9, 131.7)
- added R49: 22R, Resistor_SMD:R_0603_1608Metric, F.Cu at (338.9, 146.5)
- added R50: 22R, Resistor_SMD:R_0603_1608Metric, F.Cu at (352.9, 129.2)
- added R51: 22R, Resistor_SMD:R_0603_1608Metric, F.Cu at (356.9, 126.7)
- added R52: 10k, Resistor_SMD:R_0402_1005Metric, F.Cu at (426.4, 80.9)
- added R53: 10k, Resistor_SMD:R_0402_1005Metric, F.Cu at (416.0, 98.5)
- added R54: 10k, Resistor_SMD:R_0402_1005Metric, F.Cu at (403.1, 111.1)
- added R55: 10k, Resistor_SMD:R_0402_1005Metric, F.Cu at (424.6, 89.3)
- added R56: 1k, Resistor_SMD:R_0402_1005Metric, F.Cu at (420.6, 94.3)
- added R57: 1k, Resistor_SMD:R_0402_1005Metric, F.Cu at (406.6, 109.1)
- added R58: 1k, Resistor_SMD:R_0402_1005Metric, F.Cu at (411.1, 103.6)
- added R59: 1k, Resistor_SMD:R_0402_1005Metric, F.Cu at (410.6, 106.6)
- added R60: 22R, Resistor_SMD:R_0603_1608Metric, F.Cu at (412.5, 101.3)
- added R61: 22R, Resistor_SMD:R_0603_1608Metric, F.Cu at (421.2, 92.0)
- added R62: 22R, Resistor_SMD:R_0603_1608Metric, F.Cu at (407.2, 106.8)
- added R63: 22R, Resistor_SMD:R_0603_1608Metric, F.Cu at (421.2, 89.5)
- added R64: 22R, Resistor_SMD:R_0603_1608Metric, F.Cu at (425.2, 87.0)
- added R65: 22R, Resistor_SMD:R_0603_1608Metric, F.Cu at (412.5, 98.8)
- added R66: 22R, Resistor_SMD:R_0603_1608Metric, F.Cu at (416.9, 95.8)
- added R67: 22R, Resistor_SMD:R_0603_1608Metric, F.Cu at (399.6, 111.4)
- moved U1 6.52 mm to (-9.85, 15.2)
- moved L1 0.10 mm to (232.6, 84.4)
- moved R7 0.10 mm to (202.6, 87.7)
- renumbered Q4 to Q13, Q13 to Q4, R19 to R18, R18 to R19
Connections:
- R10 pad 1: Net-(R10-Pad1) -> /Dimmer channel 1/PWM1
- R4 pad 1: Net-(R4-Pad1) -> /Dimmer channel 1/PWM4
- R8 pad 1: Net-(R8-Pad1) -> /Dimmer channel 1/PWM3
- R9 pad 1: Net-(R9-Pad1) -> /Dimmer channel 1/PWM2
Routing:
- net Net-(Q10-Pad1): track 40.2 -> 10.0 mm
- net Net-(Q5-Pad3): track 40.2 -> 10.0 mm
- net Net-(Q1-Pad3): track 40.2 -> 10.0 mm
- net Net-(Q12-Pad1): track 40.1 -> 10.0 mm
- net +12V: track 39.1 -> 9.78 mm
- net Net-(Q16-Pad4): track 18.0 -> 4.50 mm
- net Net-(Q13-Pad4): track 16.8 -> 4.20 mm
- net Net-(Q3-Pad3): track 15.9 -> 3.98 mm
- net Net-(Q14-Pad4): track 15.9 -> 3.96 mm
- net Net-(Q15-Pad4): track 15.8 -> 3.94 mm
- net Net-(Q11-Pad3): track 15.7 -> 3.93 mm
- net Net-(Q4-Pad3): track 15.5 -> 3.88 mm
- net Net-(Q9-Pad3): track 15.5 -> 3.88 mm
- net Net-(Q10-Pad3): track 11.7 -> 2.94 mm
- net Net-(Q12-Pad3): track 11.6 -> 2.90 mm
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- added copper zone on B.Cu, net GND
- added copper zone on F.Cu, net GND

Commit message: Reduce solder mask clearance to 0
Other:
- rule pad_to_mask_clearance: 0.051 -> 0
Changed lines of the file:
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@@
     (pad_size 1.524 1.524)
     (pad_drill 0.762)
-    (pad_to_mask_clearance 0.051)
-    (solder_mask_min_width 0.25)
+    (pad_to_mask_clearance 0)
     (aux_axis_origin 0 0)
     (visible_elements FFFFFF7F)

Commit message: First eight channels finished
Parts:
- moved R24 291.7 mm to (196.7, 117.1), turned to 90 degrees
- moved R26 281.9 mm to (196.7, 103.5), turned to 90 degrees
- moved R30 280.2 mm to (202.6, 110.7)
- moved Q23 279.8 mm to (199.0, 109.9), turned to 270 degrees
- moved R29 277.6 mm to (202.6, 115.9), turned to 180 degrees
- moved R27 274.3 mm to (196.7, 96.7), turned to 90 degrees
- moved R31 274.1 mm to (202.6, 109.1), turned to 180 degrees
- moved R25 272.9 mm to (196.7, 110.3), turned to 90 degrees
- moved Q26 266.8 mm to (202.5, 99.7), turned to 90 degrees
- moved C31 265.6 mm to (216.0, 104.9)
- moved R34 264.8 mm to (202.6, 97.1)
- moved C26 264.5 mm to (196.7, 108.3), turned to 90 degrees
- moved Q30 264.1 mm to (208.1, 107.5)
- moved C27 263.8 mm to (196.7, 101.5), turned to 90 degrees
- moved Q20 263.8 mm to (199.0, 92.9), turned to 90 degrees
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Connections:
- net Net-(C1-Pad1) renamed /~RST
- net Net-(U3-Pad2) renamed /SCL
- net Net-(U3-Pad3) renamed /SDA
- U3 pad 8: Net-(U3-Pad8) -> +3V3
Routing:
- net Net-(Q18-Pad3): track 0.00 -> 10.0 mm
- net Net-(Q17-Pad3): track 0.00 -> 10.0 mm
- net Net-(Q19-Pad3): track 0.00 -> 10.0 mm
- net Net-(Q20-Pad3): track 0.00 -> 10.0 mm
- net +12V: track 9.78 -> 19.6 mm
- net Net-(Q32-Pad4): track 0.00 -> 4.50 mm
- net Net-(Q29-Pad4): track 0.00 -> 4.20 mm
- net Net-(Q22-Pad3): track 0.00 -> 3.98 mm
- net Net-(Q30-Pad4): track 0.00 -> 3.96 mm
- net Net-(Q31-Pad4): track 0.00 -> 3.94 mm
- net Net-(Q26-Pad3): track 0.00 -> 3.93 mm
- net Net-(Q28-Pad3): track 0.00 -> 3.88 mm
- net Net-(Q24-Pad3): track 0.00 -> 3.88 mm
- net Net-(Q25-Pad3): track 0.00 -> 2.94 mm
- net Net-(Q27-Pad3): track 0.00 -> 2.90 mm
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- added copper zone on F.Cu, net Net-(C29-Pad1)
- added copper zone on F.Cu, net Net-(C30-Pad1)
- added copper zone on F.Cu, net Net-(C31-Pad1)
- added copper zone on F.Cu, net Net-(C32-Pad1)
- added copper zone on F.Cu, net Net-(C33-Pad1)
- added copper zone on F.Cu, net Net-(C34-Pad1)
- added copper zone on F.Cu, net Net-(C35-Pad1)
- added copper zone on F.Cu, net Net-(C36-Pad1)
- added copper zone on F.Cu, net Net-(F6-Pad1)
- added copper zone on F.Cu, net Net-(F7-Pad1)
- added copper zone on F.Cu, net Net-(F8-Pad1)
- added copper zone on F.Cu, net Net-(F9-Pad1)
Other:
- board size 168.2 x 57 mm -> 168.2 x 57.6 mm

Commit message: All 16 channels layouted
Parts:
- moved F17 315.6 mm to (101.6, 114.0)
- moved C59 314.8 mm to (109.7, 104.8)
- moved F14 304.0 mm to (101.6, 95.7)
- moved C54 301.7 mm to (124.4, 104.8), turned to 180 degrees
- moved C57 300.5 mm to (93.9, 92.7), turned to 180 degrees
- moved F16 295.5 mm to (101.6, 107.8)
- moved C55 293.9 mm to (129.8, 104.8), turned to 180 degrees
- moved C60 286.5 mm to (93.9, 116.8), turned to 180 degrees
- moved R64 282.5 mm to (143.3, 105.8), turned to 180 degrees
- moved F15 281.1 mm to (101.6, 101.8)
- moved L13 280.2 mm to (113.2, 97.2), turned to 180 degrees
- moved R63 278.2 mm to (143.2, 100.7)
- moved R61 278.0 mm to (143.2, 93.8)
- moved R52 277.7 mm to (149.1, 96.7), turned to 90 degrees
- moved Q62 277.2 mm to (137.7, 102.2), turned to 180 degrees
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Routing:
- net +12V: track 19.6 -> 39.1 mm
- net Net-(Q50-Pad3): track 0.00 -> 10.0 mm
- net Net-(Q49-Pad3): track 0.00 -> 10.0 mm
- net Net-(Q33-Pad3): track 0.00 -> 10.0 mm
- net Net-(Q51-Pad3): track 0.00 -> 10.0 mm
- net Net-(Q35-Pad3): track 0.00 -> 10.0 mm
- net Net-(Q34-Pad3): track 0.00 -> 10.0 mm
- net Net-(Q52-Pad3): track 0.00 -> 10.0 mm
- net Net-(Q36-Pad3): track 0.00 -> 10.0 mm
- net Net-(Q64-Pad4): track 0.00 -> 4.50 mm
- net Net-(Q48-Pad4): track 0.00 -> 4.50 mm
- net Net-(Q61-Pad4): track 0.00 -> 4.20 mm
- net Net-(Q45-Pad4): track 0.00 -> 4.20 mm
- net Net-(Q54-Pad3): track 0.00 -> 3.98 mm
- net Net-(Q38-Pad3): track 0.00 -> 3.98 mm
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- added copper zone on F.Cu, net Net-(C41-Pad1)
- added copper zone on F.Cu, net Net-(C42-Pad1)
- added copper zone on F.Cu, net Net-(C43-Pad1)
- added copper zone on F.Cu, net Net-(C44-Pad1)
- added copper zone on F.Cu, net Net-(C45-Pad1)
- added copper zone on F.Cu, net Net-(C46-Pad1)
- added copper zone on F.Cu, net Net-(C47-Pad1)
- added copper zone on F.Cu, net Net-(C48-Pad1)
- added copper zone on F.Cu, net Net-(C53-Pad1)
- added copper zone on F.Cu, net Net-(C54-Pad1)
- added copper zone on F.Cu, net Net-(C55-Pad1)
- added copper zone on F.Cu, net Net-(C56-Pad1)
- added copper zone on F.Cu, net Net-(C57-Pad1)
- added copper zone on F.Cu, net Net-(C58-Pad1)
- added copper zone on F.Cu, net Net-(C59-Pad1)
- added copper zone on F.Cu, net Net-(C60-Pad1)
- added copper zone on F.Cu, net Net-(F10-Pad1)
- added copper zone on F.Cu, net Net-(F11-Pad1)
- added copper zone on F.Cu, net Net-(F12-Pad1)
- added copper zone on F.Cu, net Net-(F13-Pad1)
- added copper zone on F.Cu, net Net-(F14-Pad1)
- added copper zone on F.Cu, net Net-(F15-Pad1)
- added copper zone on F.Cu, net Net-(F16-Pad1)
- added copper zone on F.Cu, net Net-(F17-Pad1)
Other:
- board size 168.2 x 57.6 mm -> 167.6 x 57.6 mm

Commit message: Replace 5.08 mm pitch headers by 3.5 mm pitch
Parts:
- added J2: 12V Input, Connector_Phoenix_MC_HighVoltage:PhoenixContact_MC_1,5_2-G-5.08_1x02_P5.08mm_Horizontal, F.Cu at (153.6, 105.5)
- J3, J4, J5, J6: value Conn_01x04_Male -> Conn_01x05_Male; footprint Connector_Phoenix_MC_HighVoltage:PhoenixContact_MC_1,5_4-G-5.08_1x04_P5.08mm_Horizontal -> Connector_Wago:Wago_734-165_1x05_P3.50mm_Horizontal
- moved J1 203.7 mm to (190.1, 47.5), turned to 270 degrees
- moved U1 197.3 mm to (170.8, 94.3), turned to 45 degrees
- moved J5 0.55 mm to (93.9, 69.6)
- moved J3 0.50 mm to (251.9, 83.8)
- moved J4 0.50 mm to (251.9, 112.0)
- moved J6 0.45 mm to (93.9, 97.7)
Connections:
- J3 pad 1: Net-(F2-Pad1) -> GND
- J3 pad 2: Net-(F3-Pad1) -> Net-(F2-Pad1)
- J3 pad 3: Net-(F4-Pad1) -> Net-(F3-Pad1)
- J3 pad 4: Net-(F5-Pad1) -> Net-(F4-Pad1)
- J4 pad 1: Net-(F6-Pad1) -> GND
- J4 pad 2: Net-(F7-Pad1) -> Net-(F6-Pad1)
- J4 pad 3: Net-(F8-Pad1) -> Net-(F7-Pad1)
- J4 pad 4: Net-(F9-Pad1) -> Net-(F8-Pad1)
- J5 pad 1: Net-(F10-Pad1) -> GND
- J5 pad 2: Net-(F11-Pad1) -> Net-(F10-Pad1)
- J5 pad 3: Net-(F12-Pad1) -> Net-(F11-Pad1)
- J5 pad 4: Net-(F13-Pad1) -> Net-(F12-Pad1)
- J6 pad 1: Net-(F14-Pad1) -> GND
- J6 pad 2: Net-(F15-Pad1) -> Net-(F14-Pad1)
- J6 pad 3: Net-(F16-Pad1) -> Net-(F15-Pad1)
- J6 pad 4: Net-(F17-Pad1) -> Net-(F16-Pad1)

Commit message: Layout board
Parts:
- added D1: D_Schottky, Diode_SMD:D_SOD-123, F.Cu at (160.1, 95.1)
- added F18: 500mA, Fuse:Fuse_2512_6332Metric, F.Cu at (187.1, 91.3)
- added F19: 500mA, Fuse:Fuse_2512_6332Metric, F.Cu at (167.1, 101.8)
- J2: footprint Connector_Phoenix_MC_HighVoltage:PhoenixContact_MC_1,5_2-G-5.08_1x02_P5.08mm_Horizontal -> Connector_Wago_714:Wago_714-162_1x02_P3.50mm_Horizontal
- moved C8 206.8 mm to (182.0, 113.9), turned to 270 degrees
- moved C4 198.6 mm to (177.0, 84.9)
- moved U2 193.1 mm to (181.1, 101.0), turned to 90 degrees
- moved F1 191.7 mm to (172.9, 116.4), turned to 180 degrees
- moved C5 184.6 mm to (164.4, 87.8), turned to 180 degrees
- moved C12 182.3 mm to (173.6, 102.3), turned to 270 degrees
- moved C1 181.8 mm to (165.5, 94.8), turned to 270 degrees
- moved R2 178.0 mm to (166.2, 92.8), turned to 225 degrees
- moved C2 177.1 mm to (166.3, 89.9), turned to 135 degrees
- moved Y1 173.9 mm to (163.3, 92.1), turned to 225 degrees
- moved C3 167.8 mm to (160.6, 91.3), turned to 225 degrees
- moved C7 161.3 mm to (180.4, 92.8)
- moved C9 136.8 mm to (182.5, 107.0), turned to 180 degrees
- moved C10 129.1 mm to (185.6, 103.4), turned to 90 degrees
- moved R1 125.1 mm to (164.0, 94.9), turned to 45 degrees
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Connections:
- C10 pad 1: +12V -> Net-(C10-Pad1)
- C13 pad 1: +12V -> /Dimmer channel 1/+12V
- C14 pad 1: +12V -> /Dimmer channel 1/+12V
- C15 pad 1: +12V -> /Dimmer channel 1/+12V
- C16 pad 1: +12V -> /Dimmer channel 1/+12V
- C25 pad 1: +12V -> /Dimmer channel 1/+12V
- C26 pad 1: +12V -> /Dimmer channel 1/+12V
- C27 pad 1: +12V -> /Dimmer channel 1/+12V
- C28 pad 1: +12V -> /Dimmer channel 1/+12V
- C37 pad 1: +12V -> /Dimmer channel 3/+12V
- C38 pad 1: +12V -> /Dimmer channel 3/+12V
- C39 pad 1: +12V -> /Dimmer channel 3/+12V
- C40 pad 1: +12V -> /Dimmer channel 3/+12V
- C49 pad 1: +12V -> /Dimmer channel 3/+12V
- C50 pad 1: +12V -> /Dimmer channel 3/+12V
- C51 pad 1: +12V -> /Dimmer channel 3/+12V
- C52 pad 1: +12V -> /Dimmer channel 3/+12V
- C8 pad 1: +12V -> Net-(C10-Pad1)
- C9 pad 1: +12V -> Net-(C10-Pad1)
- F1 pad 1: +12V -> Net-(C10-Pad1)
- F1 pad 2: Net-(F1-Pad2) -> +12V
- J2 pad 1: Net-(F1-Pad2) -> +12V
- Q10 pad 2: +12V -> /Dimmer channel 1/+12V
- Q12 pad 2: +12V -> /Dimmer channel 1/+12V
- Q2 pad 2: +12V -> /Dimmer channel 1/+12V
- Q21 pad 2: +12V -> /Dimmer channel 1/+12V
- Q23 pad 2: +12V -> /Dimmer channel 1/+12V
- Q25 pad 2: +12V -> /Dimmer channel 1/+12V
- Q27 pad 2: +12V -> /Dimmer channel 1/+12V
- Q37 pad 2: +12V -> /Dimmer channel 3/+12V
- Q39 pad 2: +12V -> /Dimmer channel 3/+12V
- Q41 pad 2: +12V -> /Dimmer channel 3/+12V
- Q43 pad 2: +12V -> /Dimmer channel 3/+12V
- Q53 pad 2: +12V -> /Dimmer channel 3/+12V
- Q55 pad 2: +12V -> /Dimmer channel 3/+12V
- Q57 pad 2: +12V -> /Dimmer channel 3/+12V
- Q59 pad 2: +12V -> /Dimmer channel 3/+12V
- Q8 pad 2: +12V -> /Dimmer channel 1/+12V
- R10 pad 1: /Dimmer channel 1/PWM1 -> /PWM3
- R11 pad 2: +12V -> /Dimmer channel 1/+12V
- R12 pad 2: +12V -> /Dimmer channel 1/+12V
- R13 pad 2: +12V -> /Dimmer channel 1/+12V
- R20 pad 1: /Dimmer channel 2/PWM4 -> /PWM8
- R21 pad 1: /Dimmer channel 2/PWM3 -> /PWM9
- R22 pad 1: /Dimmer channel 2/PWM2 -> /PWM10
- R23 pad 1: /Dimmer channel 2/PWM1 -> /PWM11
- R24 pad 2: +12V -> /Dimmer channel 1/+12V
- R25 pad 2: +12V -> /Dimmer channel 1/+12V
- R26 pad 2: +12V -> /Dimmer channel 1/+12V
- R27 pad 2: +12V -> /Dimmer channel 1/+12V
- R36 pad 1: /Dimmer channel 3/PWM4 -> /PWM12
- R37 pad 1: /Dimmer channel 3/PWM3 -> /PWM13
- R38 pad 1: /Dimmer channel 3/PWM2 -> /PWM14
- R39 pad 1: /Dimmer channel 3/PWM1 -> /PWM15
- R4 pad 1: /Dimmer channel 1/PWM4 -> /PWM0
- R40 pad 2: +12V -> /Dimmer channel 3/+12V
- R41 pad 2: +12V -> /Dimmer channel 3/+12V
- R42 pad 2: +12V -> /Dimmer channel 3/+12V
- R43 pad 2: +12V -> /Dimmer channel 3/+12V
- R5 pad 2: +12V -> /Dimmer channel 1/+12V
- R52 pad 1: /Dimmer channel 4/PWM4 -> /PWM4
- R53 pad 1: /Dimmer channel 4/PWM3 -> /PWM5
- R54 pad 1: /Dimmer channel 4/PWM2 -> /PWM6
- R55 pad 1: /Dimmer channel 4/PWM1 -> /PWM7
- R56 pad 2: +12V -> /Dimmer channel 3/+12V
- R57 pad 2: +12V -> /Dimmer channel 3/+12V
- R58 pad 2: +12V -> /Dimmer channel 3/+12V
- R59 pad 2: +12V -> /Dimmer channel 3/+12V
- R8 pad 1: /Dimmer channel 1/PWM3 -> /PWM1
- R9 pad 1: /Dimmer channel 1/PWM2 -> /PWM2
- U1 pad 10: Net-(U1-Pad10) -> /PWM4
- U1 pad 11: Net-(U1-Pad11) -> /PWM5
- U1 pad 12: Net-(U1-Pad12) -> /PWM6
- U1 pad 13: Net-(U1-Pad13) -> /PWM7
- U1 pad 16: Net-(U1-Pad16) -> /PWM8
- U1 pad 17: Net-(U1-Pad17) -> /PWM9
- U1 pad 18: Net-(U1-Pad18) -> /PWM10
- U1 pad 19: Net-(U1-Pad19) -> /PWM11
- U1 pad 21: Net-(U1-Pad21) -> /SCL
- U1 pad 22: Net-(U1-Pad22) -> /SDA
- U1 pad 29: Net-(U1-Pad29) -> /PWM0
- U1 pad 30: Net-(U1-Pad30) -> /PWM1
- U1 pad 31: Net-(U1-Pad31) -> /PWM2
- U1 pad 32: Net-(U1-Pad32) -> /PWM3
- U1 pad 42: Net-(U1-Pad42) -> /PWM12
- U1 pad 43: Net-(U1-Pad43) -> /PWM13
- U1 pad 45: Net-(U1-Pad45) -> /PWM14
- U1 pad 46: Net-(U1-Pad46) -> /PWM15
- U2 pad 3: +12V -> Net-(C10-Pad1)
- U3 pad 2: /SCL -> GND
- U3 pad 4: (no net) -> /SCL
Routing:
- net +3V3: track 0.00 -> 86.6 mm, vias 0 -> 9
- net /Dimmer channel 3/+12V: track 0.00 -> 43.0 mm, vias 0 -> 20
- net /PWM3: track 0.00 -> 41.8 mm
- net /PWM7: track 0.00 -> 40.8 mm
- net /PWM8: track 0.00 -> 37.8 mm
- net /PWM12: track 0.00 -> 36.6 mm
- net /PWM2: track 0.00 -> 35.3 mm
- net /SWDIO: track 0.00 -> 34.2 mm, vias 0 -> 4
- net /SWCLK: track 0.00 -> 33.8 mm, vias 0 -> 4
- net /PWM6: track 0.00 -> 32.7 mm
- net /Dimmer channel 1/+12V: track 0.00 -> 31.4 mm, vias 0 -> 20
- net /PWM9: track 0.00 -> 31.2 mm
- net /PWM13: track 0.00 -> 30.0 mm
- net /PWM1: track 0.00 -> 29.2 mm
- net /PWM4: track 0.00 -> 27.6 mm
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- added copper zone on F.Cu, net +12V
- added copper zone on F.Cu, net +3V3
- added copper zone on B.Cu, net /Dimmer channel 1/+12V
- added copper zone on B.Cu, net /Dimmer channel 3/+12V
Other:
- board text added: "+ -"
- board text added: "12V PWR"
