File: dimmer_channel.sch (KiCad schematic (older format))
At the start: 53 parts, among them J3 Conn_01x04_Male, Q1 S9013, Q10 BSS84, Q11 2N7002, Q12 BSS84, Q13 VS5810AS, Q14 VS5810AS, Q15 VS5810AS, Q16 VS5810AS, Q2 BSS84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

Commit message: Replace 5.08 mm pitch headers by 3.5 mm pitch
Parts:
- J3: value Conn_01x04_Male -> Conn_01x05_Male; footprint Connector_Phoenix_MC_HighVoltage:PhoenixContact_MC_1,5_4-G-5.08_1x04_P5.08mm_Horizontal -> Connector_Wago:Wago_734-165_1x05_P3.50mm_Horizontal; symbol Connector:Conn_01x04_Male -> Connector:Conn_01x05_Male
Connections:
- wire segments 126 -> 130
