File: HB-LC-DimPWM-PCB.sch (KiCad schematic (older format))
At the start: 29 parts, among them J1 SWD, J2 12V Input, U1 STM32F103C8Tx, U2 AMS1117-3.3, U3 HomeMatic-sensor, Y1 8MHz

Commit message: Add metadata to schematic
Parts:
- U3: symbol HomeMatic-sensor:HomeMatic-sensor -> HB-LC-DimPWM-PCB-rescue:HomeMatic-sensor-HomeMatic-sensor-HB-LC-DimPWM-PCB-rescue
Changed lines of the file:
@@
 encoding utf-8
 Sheet 1 5
-Title ""
-Date ""
-Rev ""
-Comp ""
+Title "HB-LC-DimPWM"
+Date "2020-04-05"
+Rev "A"
+Comp "Tobias Schramm / Tobias Mädel"
 Comment1 ""
 Comment2 ""
@@
 	2150 2750 2050 2750
 $Comp
-L HomeMatic-sensor:HomeMatic-sensor U3
+L HB-LC-DimPWM-PCB-rescue:HomeMatic-sensor-HomeMatic-sensor-HB-LC-DimPWM-PCB-rescue U3
 U 1 1 5E9FF214
 P 5650 6150

Commit message: Remove rescue lib
Parts:
- U3: symbol HB-LC-DimPWM-PCB-rescue:HomeMatic-sensor-HomeMatic-sensor-HB-LC-DimPWM-PCB-rescue -> HomeMatic-sensor:HomeMatic-sensor
Changed lines of the file:
@@
 	2150 2750 2050 2750
 $Comp
-L HB-LC-DimPWM-PCB-rescue:HomeMatic-sensor-HomeMatic-sensor-HB-LC-DimPWM-PCB-rescue U3
+L HomeMatic-sensor:HomeMatic-sensor U3
 U 1 1 5E9FF214
 P 5650 6150

Commit message: Add tooling holes
Parts:
- added H1, H2: ToolingHole, ToolingHole:ToolingHole_JLCSMT, symbol Mechanical:MountingHole
Changed lines of the file:
@@
 	8900 1550 9000 1550
 Connection ~ 9350 1550
+$Comp
+L Mechanical:MountingHole H1
+U 1 1 5E8AC18C
+P 10550 650
+F 0 "H1" H 10650 696 50  0000 L CNN
+F 1 "ToolingHole" H 10650 605 50  0000 L CNN
+F 2 "ToolingHole:ToolingHole_JLCSMT" H 10550 650 50  0001 C CNN
+F 3 "~" H 10550 650 50  0001 C CNN
+	1    10550 650
+	1    0    0    -1
+$EndComp
+$Comp
+L Mechanical:MountingHole H2
+U 1 1 5E8AC9BB
+P 10550 900
+F 0 "H2" H 10650 946 50  0000 L CNN
+F 1 "ToolingHole" H 10650 855 50  0000 L CNN
+F 2 "ToolingHole:ToolingHole_JLCSMT" H 10550 900 50  0001 C CNN
+F 3 "~" H 10550 900 50  0001 C CNN
+	1    10550 900
+	1    0    0    -1
+$EndComp
 $EndSCHEMATC
